File: board/oval_v5.kicad_pcb (KiCad board)
At the start: 2 copper layers, 40 x 65 mm, 85 parts, among them J1 Conn_01x08, J10 HDR-4x1, J11 HDR-4x1, J13 HDR-4x1, J14 HDR-4x1, J15 HDR-4x1, J16 HDR-2x1, J2 HDR-4x1, J3 HDR-4x1, J4 Raspberry_Pi_2_3, J5 HDR-4x1, J6 HDR-4x1, J7 HDR-5x1, J8 HDR-4x1, J9 HDR-4x1, Q1 MMBT3904

Commit message: starting layout
Parts:
- removed G***: LOGO, IoWLabsLogos:cinnda
- removed G***: LOGO, IoWLabsLogos:TEDS
- removed G***: LOGO, IoWLabsLogos:cinnda_2
- removed kibuzzard-67C8B814 (x9): G***, kibuzzard-67C8B814
- removed kibuzzard-67C8B820 (x12): G***, kibuzzard-67C8B820
- removed kibuzzard-67C8B833 (x9): G***, kibuzzard-67C8B833
- removed kibuzzard-67C8B83B (x12): G***, kibuzzard-67C8B83B
- removed kibuzzard-67C8B8FE (x2): G***, kibuzzard-67C8B8FE
- removed kibuzzard-67C8B921: G***, kibuzzard-67C8B921
- removed kibuzzard-67C9C41C: G***, kibuzzard-67C9C41C
- removed kibuzzard-67C9E2A8: G***, kibuzzard-67C9E2A8
- removed kibuzzard-67C9E2B2: G***, kibuzzard-67C9E2B2
- removed kibuzzard-67C9E2C6: G***, kibuzzard-67C9E2C6
- removed kibuzzard-67C9E354: G***, kibuzzard-67C9E354
- removed kibuzzard-67C9E4BC: G***, kibuzzard-67C9E4BC
- removed kibuzzard-67C9F52F: G***, kibuzzard-67C9F52F
- removed kibuzzard-67C9F53E: G***, kibuzzard-67C9F53E
- removed kibuzzard-67C9F55A: G***, kibuzzard-67C9F55A
- removed kibuzzard-67CAE5B4 (x7): G***, kibuzzard-67CAE5B4
- removed kibuzzard-67CAE5FB: G***, kibuzzard-67CAE5FB
- added BT1: Battery_Cell, Battery:BatteryHolder_Keystone_3000_1x12mm, B.Cu at (117.5, 57.4)
- added C1: 10n, Capacitor_SMD:C_0603_1608Metric, F.Cu at (173.8, 56.1)
- added C10: 4.7u, Capacitor_SMD:C_0805_2012Metric, F.Cu at (175.5, 94.2)
- added C11: 100n, Capacitor_SMD:C_0603_1608Metric, F.Cu at (173.8, 71.1)
- added C12: 100n, Capacitor_SMD:C_0603_1608Metric, F.Cu at (173.8, 73.6)
- added C13: 1n, Capacitor_SMD:C_0603_1608Metric, F.Cu at (173.8, 76.1)
- added C14: 100n, Capacitor_SMD:C_0603_1608Metric, F.Cu at (173.8, 78.7)
- added C15: 100n, Capacitor_SMD:C_0603_1608Metric, F.Cu at (177.8, 56.1)
- added C16: 10u, Capacitor_SMD:C_0805_2012Metric, F.Cu at (63.6, 97.2)
- added C17: 10u, Capacitor_SMD:C_0805_2012Metric, F.Cu at (75.3, 97.8)
- added C18: 22u, Capacitor_SMD:C_0805_2012Metric, F.Cu at (73.3, 97.8)
- added C19: 22u, Capacitor_SMD:C_0805_2012Metric, F.Cu at (84.5, 97.8)
- added C2: 10u, Capacitor_SMD:C_0805_2012Metric, F.Cu at (175.5, 85.1)
- added C20: 1uf, Capacitor_SMD:C_0805_2012Metric, F.Cu at (184.4, 85.1)
- added C21: 1uf, Capacitor_SMD:C_0805_2012Metric, F.Cu at (184.4, 88.1)
- added C22: 1uf, Capacitor_SMD:C_0805_2012Metric, F.Cu at (184.4, 91.2)
- added C23: 1uf, Capacitor_SMD:C_0805_2012Metric, F.Cu at (184.4, 94.2)
- added C24: 100n, Capacitor_SMD:C_0603_1608Metric, F.Cu at (177.8, 58.6)
- added C25: 100n, Capacitor_SMD:C_0603_1608Metric, F.Cu at (177.8, 61.1)
- added C26: 100n, Capacitor_SMD:C_0603_1608Metric, F.Cu at (177.8, 63.6)
- added C27: 100n, Capacitor_SMD:C_0603_1608Metric, F.Cu at (177.8, 66.1)
- added C28: 100n, Capacitor_SMD:C_0603_1608Metric, F.Cu at (177.8, 68.6)
- added C29: 1uf, Capacitor_SMD:C_0805_2012Metric, F.Cu at (109.0, 110.9)
- added C3: 100n, Capacitor_SMD:C_0603_1608Metric, F.Cu at (173.8, 58.6)
- added C30: 100n, Capacitor_SMD:C_0603_1608Metric, F.Cu at (108.8, 124.6)
- added C31: 1uf, Capacitor_SMD:C_0805_2012Metric, F.Cu at (109.0, 114.0)
- added C32: 100n, Capacitor_SMD:C_0603_1608Metric, F.Cu at (108.8, 127.1)
- added C4: 100n, Capacitor_SMD:C_0603_1608Metric, F.Cu at (173.8, 61.1)
- added C5: 100n, Capacitor_SMD:C_0603_1608Metric, F.Cu at (127.8, 57.5)
- added C6: 100n, Capacitor_SMD:C_0603_1608Metric, F.Cu at (132.1, 57.5)
- added C8: 100n, Capacitor_SMD:C_0603_1608Metric, F.Cu at (173.8, 68.6)
- added C9: 10u, Capacitor_SMD:C_0805_2012Metric, F.Cu at (175.5, 91.2)
- added D10: WS2812B, LED_SMD:LED_WS2812B_PLCC4_5.0x5.0mm_P3.2mm, F.Cu at (130.1, 96.8)
- added D2: LESD5D5.0CT1G, Diode_SMD:D_SOD-523, F.Cu at (105.6, 88.9)
- added D3: LESD5D5.0CT1G, Diode_SMD:D_SOD-523, F.Cu at (108.0, 88.9)
- added D4: LESD5D5.0CT1G, Diode_SMD:D_SOD-523, F.Cu at (110.5, 88.9)
- added D5: 1N5819WS, Diode_SMD:D_SOD-323, F.Cu at (102.7, 86.2)
- added D6: LED, LED_SMD:LED_0603_1608Metric, F.Cu at (81.9, 80.2)
- added D7: D_Schottky, Diode_SMD:D_SMA, F.Cu at (122.8, 93.8)
- added D8: 1N4148W, Diode_SMD:D_SOD-123, F.Cu at (71.6, 62.8)
- added D9: 1N4148W, Diode_SMD:D_SOD-123, F.Cu at (75.1, 63.2)
- added F1: Fuse, Fuse:Fuse_1206_3216Metric, F.Cu at (118.1, 97.5)
- added J12: HDR-4x1, Connector_JST:JST_SH_BM04B-SRSS-TB_1x04-1MP_P1.00mm_Vertical, F.Cu at (52.7, 80.1)
- added J17: HDR-4x1, Connector_JST:JST_SH_BM04B-SRSS-TB_1x04-1MP_P1.00mm_Vertical, F.Cu at (57.9, 89.5)
- added J18: Conn_Coaxial, Connector_Coaxial:U.FL_Molex_MCRF_73412-0110_Vertical, F.Cu at (107.8, 52.9)
- added J19: Conn_01x02, Connector_Wago:Wago_734-132_1x02_P3.50mm_Vertical, F.Cu at (92.7, 95.0)
- added J20: Conn_01x02, Connector_PinHeader_2.54mm:PinHeader_1x02_P2.54mm_Vertical, F.Cu at (143.3, 124.2)
- added J21: Conn_02x02_Counter_Clockwise, Connector_PinHeader_2.54mm:PinHeader_2x02_P2.54mm_Vertical, F.Cu at (138.6, 131.4)
- added J22: HDR-2x1, Connector_JST:JST_XH_B2B-XH-A_1x02_P2.50mm_Vertical, F.Cu at (74.3, 53.1)
- added J23: HDR-2x1, Connector_JST:JST_XH_B2B-XH-A_1x02_P2.50mm_Vertical, F.Cu at (65.2, 53.2)
- added J25: Conn_01x06, Connector_PinHeader_2.54mm:PinHeader_1x06_P2.54mm_Vertical, F.Cu at (104.5, 111.8)
- added MK1: ICS-43434, Sensor_Audio:InvenSense_ICS-43434-6_3.5x2.65mm, F.Cu at (112.5, 73.6)
- added P1: USB_C_Plug_USB2.0, Connector_USB:USB_C_Receptacle_GCT_USB4105-xx-A_16P_TopMnt_Horizontal, F.Cu at (108.0, 96.9)
- added Q2: MMBT3904, Package_TO_SOT_SMD:SOT-23, F.Cu at (67.3, 59.2)
- added Q3: MMBT3904, Package_TO_SOT_SMD:SOT-23, F.Cu at (79.2, 60.0)
- added R10: 2.2k, Resistor_SMD:R_0603_1608Metric, F.Cu at (181.8, 68.6)
- added R11: 2.2k, Resistor_SMD:R_0603_1608Metric, F.Cu at (181.8, 71.1)
- added R12: 10k, Resistor_SMD:R_0603_1608Metric, F.Cu at (181.8, 73.6)
- added R13: 4.7k, Resistor_SMD:R_0603_1608Metric, F.Cu at (181.8, 76.1)
- added R14: 4.7k, Resistor_SMD:R_0603_1608Metric, F.Cu at (181.8, 78.7)
- added R15: 330, Resistor_SMD:R_0603_1608Metric, F.Cu at (185.8, 56.1)
- added R16: 10K, Resistor_SMD:R_0603_1608Metric, F.Cu at (185.8, 58.6)
- added R17: 10K, Resistor_SMD:R_0603_1608Metric, F.Cu at (185.8, 61.1)
- added R18: 10k, Resistor_SMD:R_0603_1608Metric, F.Cu at (185.8, 63.6)
- added R19: 10k, Resistor_SMD:R_0603_1608Metric, F.Cu at (185.8, 66.1)
- added R20: 120, Resistor_SMD:R_0603_1608Metric, F.Cu at (185.8, 68.6)
- added R21: 1k, Resistor_SMD:R_0603_1608Metric, F.Cu at (185.8, 71.1)
- added R22: 1k, Resistor_SMD:R_0603_1608Metric, F.Cu at (185.8, 73.6)
- added R23: 10k, Resistor_SMD:R_0603_1608Metric, F.Cu at (185.8, 76.1)
- added R24: 10k, Resistor_SMD:R_0603_1608Metric, F.Cu at (185.8, 78.7)
- added R25: 1k, Resistor_SMD:R_0603_1608Metric, F.Cu at (189.8, 56.1)
- added R26: 10k, Resistor_SMD:R_0603_1608Metric, F.Cu at (189.8, 58.6)
- added R27: 10k, Resistor_SMD:R_0603_1608Metric, F.Cu at (189.8, 61.1)
- added R28: 10k, Resistor_SMD:R_0603_1608Metric, F.Cu at (189.8, 63.6)
- added R29: 10k, Resistor_SMD:R_0603_1608Metric, F.Cu at (189.8, 66.1)
- added R3: 3.3k, Resistor_SMD:R_0603_1608Metric, F.Cu at (177.8, 76.1)
- added R30: 100k, Resistor_SMD:R_0603_1608Metric, F.Cu at (189.8, 68.6)
- added R4: 3.3k, Resistor_SMD:R_0603_1608Metric, F.Cu at (177.8, 78.7)
- added R5: 3.3k, Resistor_SMD:R_0603_1608Metric, F.Cu at (181.8, 56.1)
- added R6: 10K, Resistor_SMD:R_0603_1608Metric, F.Cu at (126.2, 57.5)
- added R7: 100k, Resistor_SMD:R_0603_1608Metric, F.Cu at (181.8, 61.1)
- added R8: 10K, Resistor_SMD:R_0603_1608Metric, F.Cu at (130.6, 57.5)
- added R9: 100k, Resistor_SMD:R_0603_1608Metric, F.Cu at (181.8, 66.1)
- added SW1: SW_DIP_x02, IoWLabs:SMD_SWITCH, F.Cu at (125.1, 51.9)
- added SW2: SW_DIP_x02, IoWLabs:SMD_SWITCH, F.Cu at (132.5, 51.8)
- added U1: RV-8803, IoWLabs:SON-8, B.Cu at (130.4, 58.5)
- added U10: SiP32431DR3, Package_TO_SOT_SMD:SOT-363_SC-70-6, F.Cu at (76.1, 84.5)
- added U11: SiP32431DR3, Package_TO_SOT_SMD:SOT-363_SC-70-6, F.Cu at (80.4, 84.7)
- added U12: SiP32431DR3, Package_TO_SOT_SMD:SOT-363_SC-70-6, F.Cu at (84.8, 87.8)
- added U13: SiP32431DR3, Package_TO_SOT_SMD:SOT-363_SC-70-6, F.Cu at (84.8, 84.6)
- added U14: SiP32431DR3, Package_TO_SOT_SMD:SOT-363_SC-70-6, F.Cu at (76.1, 88.0)
- added U15: PCF8574TS, Package_SO:SSOP-20_4.4x6.5mm_P0.65mm, F.Cu at (65.7, 85.1)
- added U16: PCA9548APW, Package_SO:TSSOP-24_4.4x7.8mm_P0.65mm, F.Cu at (65.6, 75.6)
- added U17: SiP32431DR3, Package_TO_SOT_SMD:SOT-363_SC-70-6, F.Cu at (80.4, 88.0)
- added U2: ESP32-S3-WROOM-1, RF_Module:ESP32-S3-WROOM-1, F.Cu at (132.1, 75.0)
- added U3: TMP117xxDRV, Package_SON:WSON-6-1EP_2x2mm_P0.65mm_EP1x1.6mm, F.Cu at (98.4, 75.7)
- added U4: RFM95W-915S2, RF_Module:HOPERF_RFM9XW_SMD, B.Cu at (96.1, 59.4)
- added U5: ~, IoWLabs:C-TQFN12-4.0x3.7-1, F.Cu at (107.9, 73.5)
- added U6: ~, IoWLabs:WSOF6I, F.Cu at (107.6, 77.9)
- added U7: MAX3485, Package_SO:SOP-8_3.9x4.9mm_P1.27mm, F.Cu at (200.8, 69.7)
- added U8: AP7361C-33E, Package_TO_SOT_SMD:SOT-223-3_TabPin2, F.Cu at (68.7, 95.2)
- added U9: AP7361C-33E, Package_TO_SOT_SMD:SOT-223-3_TabPin2, F.Cu at (80.0, 95.2)
- C7: value 100n -> 10u; footprint Capacitor_SMD:C_0603_1608Metric -> Capacitor_SMD:C_0805_2012Metric
- D1: value 1N4148W -> BAS70-05; footprint Diode_SMD:D_SOD-123 -> Package_TO_SOT_SMD:SOT-23; moved to B.Cu
- J1: value Conn_01x08 -> HDR-5x1; footprint Connector_JST:JST_GH_SM08B-GHS-TB_1x08-1MP_P1.25mm_Horizontal -> Connector_JST:JST_XH_B5B-XH-A_1x05_P2.50mm_Vertical
- J10, J11, J13, J14, J15: footprint Connector_JST:JST_XH_B4B-XH-A_1x04_P2.50mm_Vertical -> Connector_JST:JST_SH_BM04B-SRSS-TB_1x04-1MP_P1.00mm_Vertical
- J16: value HDR-2x1 -> HDR-4x1; footprint Connector_JST:JST_XH_B2B-XH-A_1x02_P2.50mm_Vertical -> Connector_JST:JST_SH_BM04B-SRSS-TB_1x04-1MP_P1.00mm_Vertical
- J4: value Raspberry_Pi_2_3 -> Conn_01x06; footprint Module:Raspberry_Pi_Zero_Socketed_THT_FaceDown_MountingHoles -> Connector_PinHeader_2.54mm:PinHeader_1x06_P2.54mm_Vertical; moved to F.Cu
- J5: value HDR-4x1 -> Micro_SD_Card; footprint Connector_JST:JST_XH_B4B-XH-A_1x04_P2.50mm_Vertical -> Connector_Card:microSD_HC_Wuerth_693072010801; moved to B.Cu
- J6: value HDR-4x1 -> Conn_01x02; footprint Connector_JST:JST_XH_B4B-XH-A_1x04_P2.50mm_Vertical -> Jumper:SolderJumper-2_P1.3mm_Open_RoundedPad1.0x1.5mm
- J7: value HDR-5x1 -> HDR-4x1; footprint Connector_JST:JST_XH_B5B-XH-A_1x05_P2.50mm_Vertical -> Connector_JST:JST_XH_B4B-XH-A_1x04_P2.50mm_Vertical
- J8: value HDR-4x1 -> Conn_01x08; footprint Connector_JST:JST_XH_B4B-XH-A_1x04_P2.50mm_Vertical -> Connector_JST:JST_GH_SM08B-GHS-TB_1x08-1MP_P1.25mm_Horizontal
- Q1: value MMBT3904 -> Q_PMOS_GSD
- R1: value 1k -> 3.3k
- R2: value 10k -> 3.3k
- moved R2 119.0 mm to (177.8, 73.6)
- moved R1 118.4 mm to (177.8, 71.1), turned to 0 degrees
- moved J1 109.2 mm to (28.8, 160.9), turned to 0 degrees
- moved C7 101.3 mm to (175.5, 88.1)
- moved J2 79.0 mm to (15.3, 129.1), turned to 0 degrees
- moved J3 75.7 mm to (15.3, 136.9), turned to 0 degrees
- moved J6 69.6 mm to (118.8, 138.0), turned to 0 degrees
- moved J9 68.9 mm to (31.1, 137.2), turned to 0 degrees
- moved D1 66.5 mm to (135.2, 56.8), turned to 90 degrees
- moved Q1 63.3 mm to (118.3, 87.9)
- moved J8 62.2 mm to (33.7, 150.8), turned to 0 degrees
- moved J5 57.8 mm to (128.8, 94.7), turned to 0 degrees
- moved J4 53.4 mm to (51.6, 159.9), turned to 90 degrees
- moved J7 43.0 mm to (31.1, 129.4), turned to 0 degrees
- moved J16 36.1 mm to (57.9, 79.9), turned to 90 degrees
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Connections:
- C7 pad 1: +3.3V -> GND
- C7 pad 2: GND -> /V_USB
- D1 pad 1: +5V -> V_DL
- D1 pad 2: FAN_- -> V_DL
- J1 pad 1: unconnected-(J1-Pin_1-Pad1) -> V_S2
- J1 pad 2: unconnected-(J1-Pin_2-Pad2) -> GND
- J1 pad 3: +3.3V -> SCL
- J1 pad 4: S_TXD -> SDA
- J1 pad 5: S_RXD -> CJ
- J10 pad 1: +3.3V -> GND
- J10 pad 2: GND -> V_S2
- J10 pad 3: RX_1 -> SDA_0
- J10 pad 4: TX_1 -> SCL_0
- J11 pad 1: +3.3V -> GND
- J11 pad 2: GND -> V_S2
- J11 pad 3: SCL -> SDA_2
- J11 pad 4: SDA -> SCL_2
- J13 pad 1: +3.3V -> GND
- J13 pad 2: GND -> V_S2
- J13 pad 3: RX_3 -> SDA_6
- J13 pad 4: TX_3 -> SCL_6
- J14 pad 1: +3.3V -> GND
- J14 pad 2: GND -> V_S2
- J14 pad 3: RX_4 -> SDA_1
- J14 pad 4: TX_4 -> SCL_1
- J15 pad 1: +3.3V -> GND
- J15 pad 2: GND -> V_S2
- J15 pad 3: SCL -> SDA_3
- J15 pad 4: SDA -> SCL_3
- J16 pad 1: +5V -> GND
- J16 pad 2: FAN_- -> V_S2
- J2 pad 1: +3.3V -> GND
- J2 pad 2: GND -> V_S2
- J2 pad 3: SCL -> SDA
- J2 pad 4: SDA -> SCL
- J3 pad 1: +3.3V -> GND
- J3 pad 2: GND -> unconnected-(J3-Pad2)
- J3 pad 3: SCL -> SDA
- J3 pad 4: SDA -> SCL
- J4 pad 1: +3.3V -> V_S2
- J4 pad 2: +5V -> GND
- J4 pad 4: +5V -> SCL
- J4 pad 5: SCL -> GND
- J4 pad 6: GND -> V_S2
- J5 pad 1: +3.3V -> unconnected-(J5-DAT2-Pad1)
- J5 pad 2: GND -> Net-(J5-DAT3/CD)
- J5 pad 3: SCL -> Net-(J5-CMD)
- J5 pad 4: SDA -> V_DL
- J6 pad 1: +3.3V -> /EVI
- J7 pad 1: +3.3V -> /RS485_B
- J7 pad 2: GND -> /RS485_A
- J7 pad 3: SCL -> GND
- J7 pad 4: SDA -> +5V
- J8 pad 1: +3.3V -> unconnected-(J8-Pin_1-Pad1)
- J8 pad 2: GND -> unconnected-(J8-Pin_2-Pad2)
- J8 pad 3: SCL -> V_S2
- J8 pad 4: SDA -> S_TXD
- J9 pad 1: +3.3V -> /RS485_B
- J9 pad 2: GND -> /RS485_A
- J9 pad 3: SCL -> GND
- J9 pad 4: SDA -> +5V
- Q1 pad 1: Net-(Q1-B) -> VIN_5V
- Q1 pad 2: GND -> 5V_VDD
- Q1 pad 3: FAN_- -> /V_USB
- R1 pad 1: Net-(Q1-B) -> Net-(D1-K)
- R1 pad 2: EN_FAN -> Net-(BT1-+)
- R2 pad 1: GND -> SD_CS
- R2 pad 2: Net-(Q1-B) -> Net-(J5-DAT3/CD)
Routing:
- net +3.3V: track 184.4 -> 0.00 mm, vias 2 -> 0
- net +5V: track 128.3 -> 0.00 mm, vias 1 -> 0
- net SCL: track 91.5 -> 0.00 mm
- net SDA: track 89.1 -> 0.00 mm
- net S_RXD: track 58.4 -> 0.00 mm
- net S_TXD: track 52.4 -> 0.00 mm
- net TX_1: track 28.3 -> 0.00 mm
- net GND: track 26.9 -> 0.00 mm, vias 18 -> 0
- net TX_4: track 26.6 -> 0.00 mm
- net FAN_-: track 26.6 -> 0.00 mm
- net RX_1: track 25.7 -> 0.00 mm
- net CJ: track 23.4 -> 0.00 mm
- net RX_4: track 21.3 -> 0.00 mm
- net RX_3: track 15.4 -> 0.00 mm
- net TX_3: track 12.8 -> 0.00 mm
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- removed copper zone on B.Cu, net GND
- removed copper zone on F.Cu, net GND
Other:
- board size 40 x 65 mm -> 95 x 50 mm

Commit message: commponent placement finished
Parts:
- removed J2: HDR-4x1, Connector_JST:JST_XH_B4B-XH-A_1x04_P2.50mm_Vertical
- removed J21: Conn_02x02_Counter_Clockwise, Connector_PinHeader_2.54mm:PinHeader_2x02_P2.54mm_Vertical
- C1, C10, C2, C20, C21, C22, C23, C25, C26, C27, C28, C29, C3, C30, C31, C32, J6, R1, R10, R11, R12, R2, R3, R4, R5, R7, R9, U10, U11, U12, U13, U14, U17: moved to B.Cu
- moved R22 120.9 mm to (65.3, 63.6), turned to -90 degrees
- moved J8 119.0 mm to (102.5, 53.7), turned to 180 degrees
- moved R24 118.7 mm to (67.9, 64.4), turned to 180 degrees
- moved C4 117.1 mm to (57.4, 73.8), turned to 180 degrees
- moved R21 111.8 mm to (74.2, 63.6), turned to -90 degrees
- moved U7 111.5 mm to (89.3, 71.0), turned to 90 degrees
- moved R23 109.5 mm to (76.9, 64.5), turned to 180 degrees
- moved R26 104.4 mm to (86.9, 76.4), turned to 90 degrees
- moved C20 103.8 mm to (80.7, 81.2), turned to -90 degrees
- moved C21 103.7 mm to (80.7, 85.5), turned to -90 degrees
- moved C22 103.7 mm to (80.7, 89.7), turned to -90 degrees
- moved C23 103.7 mm to (80.8, 93.8), turned to -90 degrees
- moved R27 102.6 mm to (88.4, 76.5), turned to 90 degrees
- moved R28 100.7 mm to (89.9, 76.5), turned to 90 degrees
- moved R29 98.9 mm to (91.5, 76.5), turned to 90 degrees
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