File: board/oval_v5.kicad_pcb (KiCad board)
At the start: 4 copper layers, 100 x 60 mm, 163 parts, among them J1 HDR-5x1, J10 HDR-4x1, J11 HDR-4x1, J12 HDR-4x1, J13 HDR-4x1, J14 HDR-4x1, J15 HDR-4x1, J16 HDR-4x1, J17 HDR-4x1, J18 Conn_Coaxial, J19 Conn_01x02, J2 HDR-4x1, J20 Conn_01x02, J21 Conn_02x02_Counter_Clockwise, J22 HDR-2x1, J23 HDR-2x1, J25 Conn_01x06, J3 HDR-4x1, J4 Conn_01x06, J5 Micro_SD_Card, J6 Conn_01x02, J7 HDR-4x1, J8 Conn_01x08, J9 HDR-4x1, P1 USB_C_Plug_USB2.0, Q1 Q_PMOS_GSD, Q2 MMBT3904, Q3 MMBT3904, SW1 SW_DIP_x02, SW2 SW_DIP_x02, U1 RV-8803, U10 SiP32431DR3, U11 SiP32431DR3, U12 SiP32431DR3, U13 SiP32431DR3, U14 SiP32431DR3, U16 PCA9548APW, U17 SiP32431DR3, U18 PCA9555PW, U2 ESP32-S3-WROOM-1, U3 TMP117xxDRV, U4 RFM95W-915S2, U7 MAX3485, U8 AP7361C-33E, U9 AP7361C-33E

Commit message: generating step
Parts:
- removed kibuzzard-69963A2F: G***, kibuzzard-69963A2F
- R38, R39, R40, R41, R42, R43, R44, R45, R46, R47, R48, R49, R50, R51, R52, R53: moved to B.Cu
- moved C17 130.3 mm to (106.4, 85.7)
- moved C19 130.3 mm to (104.4, 85.7)
- moved C21 130.3 mm to (93.0, 84.2)
- moved C27 130.3 mm to (101.5, 86.8)
- moved C28 130.3 mm to (99.8, 78.6)
- moved U12 130.3 mm to (97.8, 86.8)
- moved C12 130.3 mm to (101.7, 73.2)
- moved C16 130.3 mm to (101.2, 85.8)
- moved C18 130.3 mm to (99.0, 85.8)
- moved C22 130.3 mm to (95.3, 86.9)
- moved C26 130.3 mm to (100.0, 82.8)
- moved D6 130.3 mm to (104.7, 76.7)
- moved R15 130.3 mm to (104.7, 78.4)
- moved J21 128.1 mm to (95.0, 60.4)
- moved kibuzzard-69934843 120.7 mm to (134.5, 67.1)
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Routing:
- net GSM_Tx: track 24.7 -> 19.7 mm
- net GSM_Rx: track 23.2 -> 18.5 mm, vias 1 -> 0
- net Net-(U6-DIV): track 3.28 -> 4.54 mm, vias 0 -> 1

Commit message: working on board
Parts:
- removed J16, J17: HDR-4x1, Connector_JST:JST_PH_B4B-PH-K_1x04_P2.00mm_Vertical
- removed R33: 10k, Resistor_SMD:R_0603_1608Metric
- removed U5: ~, IoWLabs:C-TQFN12-4.0x3.7-1
- removed kibuzzard-6994F1A7: G***, kibuzzard-6994F1A7
- J2, J3: footprint Connector_JST:JST_SH_BM04B-SRSS-TB_1x04-1MP_P1.00mm_Vertical -> Connector_JST:JST_SH_SM04B-SRSS-TB_1x04-1MP_P1.00mm_Horizontal
- J25: footprint Connector_JST:JST_XH_B6B-XH-A_1x06_P2.50mm_Vertical -> Connector_JST:JST_PH_B6B-PH-K_1x06_P2.00mm_Vertical
- R38, R39, R40, R41: moved to F.Cu
- moved C13 201.1 mm to (300.9, 85.9), turned to 0 degrees
- moved R19 194.9 mm to (300.9, 90.9), turned to 0 degrees
- moved C14 193.1 mm to (300.9, 88.4), turned to 0 degrees
- moved C18 127.2 mm to (225.2, 102.6)
- moved C21 127.2 mm to (219.1, 101.0)
- moved C25 127.2 mm to (209.5, 109.2)
- moved C26 127.2 mm to (226.1, 99.5)
- moved C28 127.2 mm to (225.9, 95.3)
- moved C33 127.2 mm to (198.9, 101.7)
- moved C34 127.2 mm to (198.9, 99.7)
- moved D7 127.2 mm to (215.9, 110.2)
- moved J21 127.2 mm to (221.1, 77.1)
- moved R10 127.2 mm to (196.4, 80.9)
- moved R12 127.2 mm to (252.1, 121.0)
- moved R13 127.2 mm to (240.9, 101.0)
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Connections:
- J14 pad 3: SDA_6 -> SDA_1
- J14 pad 4: SCL_6 -> SCL_1
- J15 pad 3: SDA_7 -> SDA_0
- J15 pad 4: SCL_7 -> SCL_0
Routing:
- net V_S2: track 193.2 -> 93.9 mm
- net SDA: track 37.6 -> 103.7 mm, vias 0 -> 2
- net SCL: track 37.5 -> 96.3 mm, vias 0 -> 2
- net SCL_5: track 22.9 -> 61.8 mm, vias 1 -> 4
- net GSM_PWRKEY: track 37.2 -> 0.00 mm, vias 2 -> 0
- net GSM_RST: track 37.0 -> 0.00 mm, vias 2 -> 0
- net SDA_2: track 32.2 -> 7.17 mm
- net SDA_5: track 22.9 -> 0.00 mm, vias 1 -> 0
- net SDA_6: track 20.6 -> 1.66 mm, vias 1 -> 0
- net SCL_6: track 19.4 -> 1.67 mm, vias 1 -> 0
- net GND: track 3.52 -> 20.4 mm, vias 1 -> 3
- net PMS_Rx: track 17.8 -> 1.40 mm
- net RS485_TX: track 74.7 -> 59.2 mm
- net PMS_Tx: track 17.8 -> 2.56 mm
- net RS485_RX: track 72.2 -> 57.4 mm
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Other:
- board size 100 x 60 mm -> 95 x 50 mm
