File: board/_autosave-oval_v5.kicad_pcb (KiCad board)
At the start: 2 copper layers, 95 x 50 mm, 129 parts, among them J1 HDR-5x1, J10 HDR-4x1, J11 HDR-4x1, J12 HDR-4x1, J13 HDR-4x1, J14 HDR-4x1, J15 HDR-4x1, J16 HDR-4x1, J17 HDR-4x1, J18 Conn_Coaxial, J19 Conn_01x02, J20 Conn_01x02, J22 HDR-2x1, J23 HDR-2x1, J25 Conn_01x06, J3 HDR-4x1, J4 Conn_01x06, J5 Micro_SD_Card, J6 Conn_01x02, J7 HDR-4x1, J8 Conn_01x08, J9 HDR-4x1, P1 USB_C_Plug_USB2.0, Q1 Q_PMOS_GSD, Q2 MMBT3904, Q3 MMBT3904, SW1 SW_DIP_x02, SW2 SW_DIP_x02, U1 RV-8803, U10 SiP32431DR3, U11 SiP32431DR3, U12 SiP32431DR3, U13 SiP32431DR3, U14 SiP32431DR3, U15 PCF8574TS, U16 PCA9548APW, U17 SiP32431DR3, U2 ESP32-S3-WROOM-1, U3 TMP117xxDRV, U4 RFM95W-915S2, U7 MAX3485, U8 AP7361C-33E, U9 AP7361C-33E

Commit message: minor changes
Parts:
- moved J20 0.50 mm to (107.5, 85.5)
Routing:
- net V_S2: track 85.3 -> 63.1 mm
Changed lines of the file:
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@@
 	(footprint "Connector_JST:JST_XH_B2B-XH-A_1x02_P2.50mm_Vertical"
 		(layer "F.Cu")
-		(at 107.5 85 180)
+		(at 107.5 85.5 180)
 		(descr "JST XH series connector, B2B-XH-A (http://www.jst-mfg.com/product/pdf/eng/eXH.pdf), generated with kicad-footprint-generator")
 		(tags "connector JST XH vertical")
@@
 	)
 	(segment
-		(start 58.625 91.9)
-		(end 59.35 91.175)
-		(width 0.6096)
-		(layer "B.Cu")
-		(net 12)
-	)
-	(segment
 		(start 68.775 81.75)
 		(end 68.775 84.625)
@@
 	)
 	(segment
-		(start 63.775 91.975)
-		(end 63.775 89.1)
-		(width 0.6096)
-		(layer "B.Cu")
-		(net 12)
-	)
-	(segment
-		(start 59.35 91.175)
-		(end 59.35 88.55)
-		(width 0.6096)
-		(layer "B.Cu")
-		(net 12)
-	)
-	(segment
 		(start 69.275 85.95)
 		(end 70.1 85.95)
@@
 	)
 	(segment
-		(start 53.125 91.95)
-		(end 57.125 87.95)
-		(width 0.6096)
-		(layer "B.Cu")
-		(net 12)
-	)
-	(segment
 		(start 72.675 85.95)
 		(end 76.1 89.375)
@@
 	)
 	(segment
-		(start 53.375 81.75)
-		(end 54.525 81.75)
-		(width 0.6096)
-		(layer "B.Cu")
-		(net 12)
-	)
-	(segment
 		(start 58.725 85.95)
 		(end 63.125 85.95)
@@
 	)
 	(segment
-		(start 54.525 81.75)
-		(end 57.9875 85.2125)
-		(width 0.6096)
-		(layer "B.Cu")
-		(net 12)
-	)
-	(segment
 		(start 69.25 87.9)
 		(end 71.2 85.95)
@@
 	)
 	(segment
-		(start 69.25 91.925)
-		(end 69.25 87.9)
-		(width 0.6096)
-		(layer "B.Cu")
-		(net 12)
-	)
-	(segment
 		(start 63.125 85.95)
 		(end 66.925 85.95)
@@
 	)
 	(segment
-		(start 69.95 96.75)
-		(end 69.95 97.275)
+		(start 72.25 94.075)
+		(end 70.146342 96.178658)
 		(width 0.254)
 		(layer "F.Cu")
@@
 	)
 	(segment
-		(start 90.405 85.445)
-		(end 81.255 85.445)
+		(start 93.025 83.475)
+		(end 91.055 85.445)
+		(width 0.254)
+		(layer "F.Cu")
+		(net 143)
+	)
+	(segment
+		(start 93.025 82.825)
+		(end 93.025 83.475)
+		(width 0.254)
+		(layer "F.Cu")
+		(net 143)
+	)
+	(segment
+		(start 70.146342 96.178658)
+		(end 70.146342 96.303658)
+		(width 0.254)
+		(layer "F.Cu")
+		(net 143)
+	)
+	(segment
+		(start 91.055 85.445)
+		(end 82.911532 85.445)
 		(width 0.254)
 		(layer "F.Cu")
@@
 	)
 	(segment
+		(start 82.911532 85.445)
+		(end 74.281532 94.075)
+		(width 0.254)
+		(layer "F.Cu")
+		(net 143)
+	)
+	(segment
+		(start 70.146342 96.303658)
+		(end 69.95 96.5)
+		(width 0.254)
+		(layer "F.Cu")
+		(net 143)
+	)
+	(segment
 		(start 125.965 68.985)
 		(end 125.965 66.25)
@@
 	)
 	(segment
-		(start 93.025 82.825)
-		(end 90.405 85.445)
+		(start 69.95 96.5)
+		(end 69.95 97.275)
 		(width 0.254)
 		(layer "F.Cu")
@@
 	)
 	(segment
-		(start 123.45 71.05)
-		(end 123.9 71.05)
+		(start 74.281532 94.075)
+		(end 72.25 94.075)
 		(width 0.254)
 		(layer "F.Cu")
@@
 	)
 	(segment
-		(start 81.255 85.445)
-		(end 69.95 96.75)
+		(start 123.45 71.05)
+		(end 123.9 71.05)
 		(width 0.254)
 		(layer "F.Cu")
@@
 	)
 	(segment
-		(start 94.172 83.972)
-		(end 120.495884 83.972)
+		(start 93.025 82.825)
+		(end 93.831532 82.825)
 		(width 0.254)
 		(layer "B.Cu")
@@
 	)
 	(segment
-		(start 124.522 71.872)
-		(end 123.7 71.05)
+		(start 120.926595 83.455)
+		(end 124.522 79.859594)
 		(width 0.254)
 		(layer "B.Cu")
@@
 	)
 	(segment
-		(start 124.522 79.945884)
+		(start 123.7 71.05)
+		(end 123.45 71.05)
+		(width 0.254)
+		(layer "B.Cu")
+		(net 143)
+	)
+	(segment
+		(start 124.522 79.859594)
 		(end 124.522 71.872)
 		(width 0.254)
@@
 	)
 	(segment
-		(start 120.495884 83.972)
-		(end 124.522 79.945884)
+		(start 94.461533 83.455)
+		(end 120.926595 83.455)
 		(width 0.254)
 		(layer "B.Cu")
@@
 	)
 	(segment
-		(start 93.025 82.825)
-		(end 94.172 83.972)
+		(start 93.831532 82.825)
+		(end 94.461533 83.455)
 		(width 0.254)
 		(layer "B.Cu")
@@
 	)
 	(segment
-		(start 123.7 71.05)
-		(end 123.45 71.05)
+		(start 124.522 71.872)
+		(end 123.7 71.05)
 		(width 0.254)
 		(layer "B.Cu")
@@
 	)
 	(segment
+		(start 72.45 96.55)
+		(end 72.45 97.275)
+		(width 0.254)
+		(layer "F.Cu")
+		(net 144)
+	)
+	(segment
 		(start 124.695 68.605)
 		(end 122.3 71)
@@
 	)
 	(segment
-		(start 124.65 66.205)
-		(end 124.695 66.25)
+		(start 94 83.143468)
+		(end 91.243467 85.9)
 		(width 0.254)
 		(layer "F.Cu")
@@
 	)
 	(segment
-		(start 72.45 97.275)
-		(end 72.45 94.893468)
+		(start 124.65 66.205)
+		(end 124.695 66.25)
 		(width 0.254)
 		(layer "F.Cu")
@@
 	)
 	(segment
-		(start 124.695 66.25)
-		(end 124.695 68.605)
+		(start 91.243467 85.9)
+		(end 83.1 85.9)
 		(width 0.254)
 		(layer "F.Cu")
@@
 	)
 	(segment
-		(start 94.5 83.15)
-		(end 91.75 85.9)
+		(start 94 82)
+		(end 94 83.143468)
 		(width 0.254)
 		(layer "F.Cu")
@@
 	)
 	(segment
-		(start 72.45 94.893468)
-		(end 81.443468 85.9)
+		(start 124.695 66.25)
+		(end 124.695 68.605)
 		(width 0.254)
 		(layer "F.Cu")
@@
 	)
 	(segment
-		(start 91.75 85.9)
-		(end 81.443468 85.9)
+		(start 83.1 85.9)
+		(end 72.45 96.55)
 		(width 0.254)
 		(layer "F.Cu")
@@
 	)
 	(via
-		(at 94.5 83.15)
+		(at 94 82)
 		(size 0.6)
 		(drill 0.3)
@@
 	)
 	(segment
-		(start 94.5 83.15)
-		(end 94.867 83.517)
+		(start 120.738127 83)
+		(end 124.067 79.671127)
 		(width 0.254)
 		(layer "B.Cu")
@@
 	)
 	(segment
-		(start 122.3 71)
+		(start 124.067 79.671127)
 		(end 124.067 72.767)
 		(width 0.254)
@@
 	)
 	(segment
-		(start 120.221127 83.517)
-		(end 117.7 83.517)
+		(start 94 82)
+		(end 94.075 82)
 		(width 0.254)
 		(layer "B.Cu")
@@
 	)
 	(segment
-		(start 124.067 79.671127)
-		(end 120.221127 83.517)
+		(start 94.075 82)
+		(end 95.075 83)
 		(width 0.254)
 		(layer "B.Cu")
@@
 	(segment
 		(start 124.067 72.767)
-		(end 124.067 77.767)
-		(width 0.254)
-		(layer "B.Cu")
-		(net 144)
-	)
-	(segment
-		(start 94.867 83.517)
-		(end 117.25 83.517)
-		(width 0.254)
-		(layer "B.Cu")
-		(net 144)
-	)
-	(segment
-		(start 124.067 77.767)
-		(end 124.067 79.671127)
-		(width 0.254)
-		(layer "B.Cu")
-		(net 144)
-	)
-	(segment
-		(start 117.25 83.517)
-		(end 116.851405 83.517)
+		(end 122.3 71)
 		(width 0.254)
 		(layer "B.Cu")
@@
 	)
 	(segment
-		(start 117.7 83.517)
-		(end 117.25 83.517)
+		(start 95.075 83)
+		(end 120.738127 83)
 		(width 0.254)
 		(layer "B.Cu")
