File: board/_autosave-oval_v5.kicad_sch (KiCad schematic)
At the start: 122 parts, among them J1 HDR-5x1, J10 HDR-4x1, J11 HDR-4x1, J12 HDR-4x1, J13 HDR-4x1, J14 HDR-4x1, J15 HDR-4x1, J16 HDR-4x1, J17 HDR-4x1, J18 Conn_Coaxial, J19 Conn_01x02, J2 HDR-4x1, J20 Conn_01x02, J21 Conn_02x02_Counter_Clockwise, J22 HDR-2x1, J23 HDR-2x1, J25 Conn_01x06, J3 HDR-4x1, J4 Conn_01x06, J5 Micro_SD_Card, J6 Conn_01x02, J7 HDR-4x1, J8 Conn_01x08, J9 HDR-4x1, P1 USB_C_Plug_USB2.0, Q1 Q_PMOS_GSD, Q2 MMBT3904, Q3 MMBT3904, SW1 SW_DIP_x02, SW2 SW_DIP_x02, U1 RV-8803, U10 SiP32431DR3, U11 SiP32431DR3, U12 SiP32431DR3, U13 SiP32431DR3, U14 SiP32431DR3, U15 PCF8574TS, U16 PCA9548APW, U17 SiP32431DR3, U2 ESP32-S3-WROOM-1, U3 TMP117xxDRV, U4 RFM95W-915S2, U7 MAX3485, U8 AP7361C-33E, U9 AP7361C-33E

Commit message: minor changes
Parts:
- added R31, R32, R33: 10K, Resistor_SMD:R_0603_1608Metric, symbol IoWLabs:RES
- D5: footprint Diode_SMD:D_SOD-323 -> Diode_SMD:D_SOD-323_HandSoldering
- J20: footprint Connector_PinHeader_2.54mm:PinHeader_1x02_P2.54mm_Vertical -> Connector_JST:JST_XH_B2B-XH-A_1x02_P2.50mm_Vertical
- J25, J4: footprint Connector_PinHeader_2.54mm:PinHeader_1x06_P2.54mm_Vertical -> Connector_JST:JST_XH_B6B-XH-A_1x06_P2.50mm_Vertical
Connections:
- net CLK is gone; now on net SPI_SCLK: R4.1, U4.4 (SCK)
- net MISO is gone; now on net SPI_MISO: R5.1, U4.2 (MISO)
- net MOSI is gone; now on net SPI_MOSI: R3.1, U4.3 (MOSI)
- net SIM_PWRKEY is gone; now on net GSM_PWRKEY: J25.3 (Pin_3)
- net SIM_RST is gone; now on net GSM_RST: J25.4 (Pin_4)
- net SIM_RX is gone; now on net GSM_Rx: J25.2 (Pin_2)
- net SIM_TX is gone; now on net GSM_Tx: J25.1 (Pin_1)
- net GND: now also U15.6 (A0), U15.7 (A1), U15.9 (A2), U16.1 (A0), U16.2 (A1), U16.21 (A2)
- net GSM_Rx: now also U2.10 (GPIO17/U1TXD/ADC2_CH6)
- net GSM_Tx: now also U2.11 (GPIO18/U1RXD/ADC2_CH7/CLK_OUT3)
- net RS485_EN: now also U2.25 (GPIO48/SPICLK_N/SUBSPICLK_N_DIFF)
- net SCL: now also R33.1
- net SDA: now also R32.1
- net V_L: now also R31.1, R32.2, R33.2
- net rfm_RST: now also U2.5 (GPIO5/TOUCH5/ADC1_CH4); no longer U2.10 (GPIO17/U1TXD/ADC2_CH6)
- net rfm_dio1: now also U2.24 (GPIO47/SPICLK_P/SUBSPICLK_P_DIFF); no longer U2.11 (GPIO18/U1RXD/ADC2_CH7/CLK_OUT3)
- net rfm_dio2: now also U2.6 (GPIO6/TOUCH6/ADC1_CH5), U4.16 (DIO2); no longer U2.31 (GPIO38/FSPIWP/SUBSPIWP)
- net at U16.3 (~{RESET}): now also R31.2
Other:
- note added: "Default I2C address : 0x50"
- note added: "Default I2C address : 0x70"
- moved on the sheet: J18, U4

Commit message: working on layout -  defining connectors and cables
Parts:
- added R34, R35: 10k, Resistor_SMD:R_0603_1608Metric, symbol Device:R
- added U18: PCA9555PW, Package_SO:TSSOP-24_4.4x7.8mm_P0.65mm, symbol Interface_Expansion:PCA9555PW
- J4: footprint Connector_JST:JST_XH_B6B-XH-A_1x06_P2.50mm_Vertical -> Connector_JST:JST_GH_SM06B-GHS-TB_1x06-1MP_P1.25mm_Horizontal
- J8: footprint Connector_JST:JST_GH_SM08B-GHS-TB_1x08-1MP_P1.25mm_Horizontal -> Connector_Molex:Molex_PicoBlade_53261-0871_1x08-1MP_P1.25mm_Horizontal
Connections:
- net EN_V_DL is gone; now on net V_DL_EN: U15.12 (P2)
- net EN_V_GSM is gone; now on net V_GSM_EN: U15.17 (P5)
- net EN_V_S1 is gone; now on net V_S1_EN: U15.14 (P3)
- net EN_V_S2 is gone; now on net V_S2_EN: U15.16 (P4)
- net V_S3_EN is gone; now on net V_RF_EN: U12.3 (ON)
- net +5V: now also J8.1 (Pin_1); no longer J8.8 (Pin_8)
- net GND: now also J8.2 (Pin_2); no longer J8.7 (Pin_7)
- net SCL: now also R35.2
- net SDA: now also R34.2
- net V_S2: now also R34.1, R35.1; no longer J8.3 (Pin_3)
- net EN_V_RF renamed V_RF_EN
- net S_RXD renamed PMS_Tx
- net S_TXD renamed PMS_Rx
- new net PMS_SET: J8.3 (Pin_3)
Other:
- moved on the sheet: J4, J7, J9, U15
