File: board/oval_v5 bkp.kicad_pcb (KiCad board)
At the start: 2 copper layers, 95 x 50 mm, 136 parts, among them J1 HDR-5x1, J10 HDR-4x1, J11 HDR-4x1, J12 HDR-4x1, J13 HDR-4x1, J14 HDR-4x1, J15 HDR-4x1, J16 HDR-4x1, J17 HDR-4x1, J18 Conn_Coaxial, J19 Conn_01x02, J2 HDR-4x1, J20 Conn_01x02, J21 Conn_02x02_Counter_Clockwise, J22 HDR-2x1, J23 HDR-2x1, J25 Conn_01x06, J3 HDR-4x1, J4 Conn_01x06, J5 Micro_SD_Card, J6 Conn_01x02, J7 HDR-4x1, J8 Conn_01x08, J9 HDR-4x1, P1 USB_C_Plug_USB2.0, Q1 Q_PMOS_GSD, Q2 MMBT3904, Q3 MMBT3904, SW1 SW_DIP_x02, SW2 SW_DIP_x02, U1 RV-8803, U10 SiP32431DR3, U11 SiP32431DR3, U12 SiP32431DR3, U13 SiP32431DR3, U14 SiP32431DR3, U15 PCF8574TS, U16 PCA9548APW, U17 SiP32431DR3, U2 ESP32-S3-WROOM-1, U3 TMP117xxDRV, U4 RFM95W-915S2, U7 MAX3485, U8 AP7361C-33E, U9 AP7361C-33E

Commit message: working on layout -  defining connectors and cables
Parts:
- removed kibuzzard-699C8DA6: G***, kibuzzard-699C8DA6
- removed kibuzzard-699C8DCD: G***, kibuzzard-699C8DCD
- J4: footprint Connector_JST:JST_GH_SM06B-GHS-TB_1x06-1MP_P1.25mm_Horizontal -> Connector_JST:JST_XH_B6B-XH-A_1x06_P2.50mm_Vertical
- J8: footprint Connector_Molex:Molex_PicoBlade_53261-0871_1x08-1MP_P1.25mm_Horizontal -> Connector_JST:JST_GH_SM08B-GHS-TB_1x08-1MP_P1.25mm_Horizontal
- moved J2 195.3 mm to (219.8, 63.3), turned to 0 degrees
- moved C4 128.6 mm to (60.6, 44.5), turned to 0 degrees
- moved J8 120.0 mm to (102.5, 53.7), turned to 180 degrees
- moved J4 105.7 mm to (60.0, 69.2), turned to 90 degrees
- moved J1 95.9 mm to (52.9, 69.2)
- moved J25 66.6 mm to (72.5, 97.3)
- moved U11 58.4 mm to (76.9, 87.0)
- moved J10 58.3 mm to (53.8, 78.7)
- moved J11 58.3 mm to (64.4, 78.7)
- moved J14 58.3 mm to (59.0, 78.7)
- moved J15 58.3 mm to (69.7, 78.7)
- moved J12 58.3 mm to (69.8, 88.9)
- moved J16 58.3 mm to (64.5, 88.9)
- moved kibuzzard-6993384F 58.3 mm to (73.3, 84.1)
- moved J13 58.3 mm to (59.1, 88.9)
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Routing:
- net SCL_7: track 16.8 -> 37.6 mm
- net SDA_7: track 17.4 -> 38.2 mm
- net SCL_6: track 14.9 -> 31.3 mm
- net SDA_6: track 15.7 -> 32.2 mm
- net SCL_5: track 12.8 -> 25.9 mm
- net SDA_5: track 13.6 -> 25.8 mm
- net SDA_4: track 12.3 -> 18.5 mm
- net SDA_0: track 25.8 -> 30.7 mm
- net SCL_0: track 22.7 -> 27.6 mm
- net SDA_1: track 20.5 -> 25.4 mm
- net SCL_1: track 17.6 -> 22.5 mm
- net SDA_2: track 14.9 -> 19.7 mm
- net SDA_3: track 8.79 -> 13.6 mm
- net SCL_2: track 11.6 -> 16.5 mm
- net SCL_3: track 4.51 -> 9.36 mm
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