File: board/oval_v5.kicad_sch (KiCad schematic)
At the start: 147 parts, among them J1 HDR-5x1, J10 HDR-4x1, J11 HDR-4x1, J12 HDR-4x1, J13 HDR-4x1, J14 HDR-4x1, J15 HDR-4x1, J16 HDR-4x1, J17 HDR-4x1, J18 Conn_Coaxial, J19 Conn_01x02, J2 HDR-4x1, J20 Conn_01x02, J21 Conn_02x02_Counter_Clockwise, J22 HDR-2x1, J23 HDR-2x1, J25 Conn_01x06, J3 HDR-4x1, J4 Conn_01x06, J5 Micro_SD_Card, J6 Conn_01x02, J7 HDR-4x1, J8 Conn_01x08, J9 HDR-4x1, P1 USB_C_Plug_USB2.0, Q1 Q_PMOS_GSD, Q2 MMBT3904, Q3 MMBT3904, SW1 SW_DIP_x02, SW2 SW_DIP_x02, U1 RV-8803, U10 SiP32431DR3, U11 SiP32431DR3, U12 SiP32431DR3, U13 SiP32431DR3, U14 SiP32431DR3, U16 PCA9548APW, U17 SiP32431DR3, U18 PCA9555PW, U2 ESP32-S3-WROOM-1, U3 TMP117xxDRV, U4 RFM95W-915S2, U7 MAX3485, U8 AP7361C-33E, U9 AP7361C-33E

Commit message: adding work in layout
Parts:
- R16, R17, R31, R36, R37, R38, R39, R40, R41, R42, R43, R44, R45, R46, R47, R48, R49, R50, R51, R52, R53, R6, R8: value 10K -> 10k
- R32: value 10K -> 10k; DNP| DNP -> (none)
- R33: value 10K -> 10k; DNP DNP -> (none)
Other:
- note added: "Extensores I2C"
Changed lines of the file:
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@@
 	)
 	(rectangle
+		(start 439.42 0)
+		(end 650.24 120.65)
+		(stroke
+			(width 0)
+			(type default)
+		)
+		(fill
+			(type none)
+		)
+	)
+	(rectangle
 		(start 118.11 378.46)
 		(end 223.52 441.96)
@@
 	(text "Expansor GPIO\n-------------------\nGPIO00 - onBoardLED\nGPIO01 - V_GSM_EN\nGPIO02 - V_S1_EN\nGPIO03 - V_S2_EN\nGPIO04 - V_RF_EN\nGPIO05 - V_DL_EN\nGPIO06 - FAN_1_EN\nGPIO07 - FAN_1_EN\nGPIO08 - PMS_SET\nGPIO09 - RS485_EN\nGPIO10 - I2C_BUS_RST\n\n"
 		(exclude_from_sim no)
-		(at 505.206 120.396 0)
+		(at 498.856 105.918 0)
 		(effects
 			(font
@@
 		)
 	)
+	(text "Extensores I2C"
+		(exclude_from_sim no)
+		(at 504.698 10.668 0)
+		(effects
+			(font
+				(size 4 4)
+				(thickness 0.5994)
+				(bold yes)
+			)
+			(justify left bottom)
+		)
+	)
 	(text "Auxiliar FAN drivers"
 		(exclude_from_sim no)
@@
 	(wire
 		(pts
-			(xy 635 50.8) (xy 622.3 50.8)
+			(xy 635 49.53) (xy 632.46 49.53)
 		)
 		(stroke
@@
 	(wire
 		(pts
-			(xy 635 46.99) (xy 635 50.8)
+			(xy 635 46.99) (xy 635 49.53)
 		)
 		(stroke
@@
 	(wire
 		(pts
-			(xy 629.92 45.72) (xy 629.92 48.26)
+			(xy 629.92 45.72) (xy 629.92 46.99)
 		)
 		(stroke
@@
 	(wire
 		(pts
-			(xy 629.92 48.26) (xy 622.3 48.26)
+			(xy 629.92 46.99) (xy 627.38 46.99)
 		)
 		(stroke
@@
 	(global_label "SDA"
 		(shape input)
-		(at 622.3 50.8 180)
+		(at 632.46 49.53 180)
 		(fields_autoplaced yes)
 		(effects
@@
 		)
 		(property "Intersheetrefs" "${INTERSHEET_REFS}"
-			(at 615.7467 50.8 0)
+			(at 625.9067 49.53 0)
 			(effects
 				(font
@@
 	(global_label "SCL"
 		(shape input)
-		(at 622.3 48.26 180)
+		(at 627.38 46.99 180)
 		(fields_autoplaced yes)
 		(effects
@@
 		)
 		(property "Intersheetrefs" "${INTERSHEET_REFS}"
-			(at 615.8072 48.26 0)
+			(at 620.8872 46.99 0)
 			(effects
 				(font
@@
 			)
 		)
-		(property "Value" "10K"
+		(property "Value" "10k"
 			(at 633.3236 41.91 90)
 			(effects
@@
 			)
 		)
-		(property "DNP" "DNP"
-			(at 627.38 41.91 90)
-			(effects
-				(font
-					(size 1.27 1.27)
-				)
-			)
-		)
 		(pin "1"
 		)
@@
 			)
 		)
-		(property "Value" "10K"
+		(property "Value" "10k"
 			(at 505.968 226.06 90)
 			(effects
@@
 			)
 		)
-		(property "Value" "10K"
+		(property "Value" "10k"
 			(at 578.358 226.06 90)
 			(effects
@@
 			)
 		)
-		(property "Value" "10K"
+		(property "Value" "10k"
 			(at 579.628 252.73 90)
 			(effects
@@
 			)
 		)
-		(property "Value" "10K"
+		(property "Value" "10k"
 			(at 558.038 226.314 90)
 			(effects
@@
 			)
 		)
-		(property "Value" "10K"
+		(property "Value" "10k"
 			(at 224.155 56.2864 90)
 			(effects
@@
 			)
 		)
-		(property "Value" "10K"
+		(property "Value" "10k"
 			(at 503.428 250.444 90)
 			(effects
@@
 			)
 		)
-		(property "Value" "10K"
+		(property "Value" "10k"
 			(at 560.578 226.06 90)
 			(effects
@@
 			)
 		)
-		(property "Value" "10K"
+		(property "Value" "10k"
 			(at 487.2736 38.1 90)
 			(effects
@@
 			)
 		)
-		(property "Value" "10K"
+		(property "Value" "10k"
 			(at 564.388 254 90)
 			(effects
@@
 			)
 		)
-		(property "Value" "10K"
+		(property "Value" "10k"
 			(at 77.9272 125.603 0)
 			(effects
@@
 			)
 		)
-		(property "Value" "10K"
+		(property "Value" "10k"
 			(at 503.428 226.314 90)
 			(effects
@@
 			)
 		)
-		(property "Value" "10K"
+		(property "Value" "10k"
 			(at 505.968 250.19 90)
 			(effects
@@
 			)
 		)
-		(property "Value" "10K"
+		(property "Value" "10k"
 			(at 199.39 95.6564 90)
 			(effects
@@
 			)
 		)
-		(property "Value" "10K"
+		(property "Value" "10k"
 			(at 65.2272 125.603 0)
 			(effects
@@
 			)
 		)
-		(property "Value" "10K"
+		(property "Value" "10k"
 			(at 561.848 254.254 90)
 			(effects
@@
 			)
 		)
-		(property "Value" "10K"
+		(property "Value" "10k"
 			(at 577.088 252.984 90)
 			(effects
@@
 			)
 		)
-		(property "Value" "10K"
+		(property "Value" "10k"
 			(at 575.818 226.314 90)
 			(effects
@@
 			)
 		)
-		(property "Value" "10K"
+		(property "Value" "10k"
 			(at 493.268 250.19 90)
 			(effects
@@
 			)
 		)
-		(property "Value" "10K"
+		(property "Value" "10k"
 			(at 493.268 226.06 90)
 			(effects
@@
 			)
 		)
-		(property "Value" "10K"
+		(property "Value" "10k"
 			(at 490.728 226.314 90)
 			(effects
@@
 			)
 		)
-		(property "Value" "10K"
+		(property "Value" "10k"
 			(at 482.1936 36.83 90)
 			(effects
@@
 			)
 		)
-		(property "Value" "10K"
+		(property "Value" "10k"
 			(at 638.4036 43.18 90)
 			(effects
@@
 			)
 		)
-		(property "DNP|" "DNP"
-			(at 633.222 42.926 90)
-			(effects
-				(font
-					(size 1.27 1.27)
-				)
-			)
-		)
 		(pin "1"
 		)
@@
 			)
 		)
-		(property "Datasheet" " ~"
+		(property "Datasheet" "~"
 			(at 204.47 344.17 0)
 			(effects
@@
 			)
 		)
-		(property "Value" "10K"
+		(property "Value" "10k"
 			(at 490.728 250.444 90)
 			(effects
@@
 			)
 		)
-		(property "Value" "10K"
+		(property "Value" "10k"
 			(at 565.5564 41.91 90)
 			(effects

Commit message: bom ready
Parts:
- J25: footprint Connector_JST:JST_XH_B6B-XH-A_1x06_P2.50mm_Vertical -> Connector_JST:JST_PH_B6B-PH-K_1x06_P2.00mm_Vertical
Changed lines of the file:
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@@
 			)
 		)
-		(property "Footprint" "Connector_JST:JST_XH_B6B-XH-A_1x06_P2.50mm_Vertical"
+		(property "Footprint" "Connector_JST:JST_PH_B6B-PH-K_1x06_P2.00mm_Vertical"
 			(at 59.69 463.55 0)
 			(effects

Commit message: bom already finished
Parts:
- J2, J3: footprint Connector_JST:JST_SH_BM04B-SRSS-TB_1x04-1MP_P1.00mm_Vertical -> Connector_JST:JST_SH_SM04B-SRSS-TB_1x04-1MP_P1.00mm_Horizontal
Changed lines of the file:
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@@
 			)
 		)
-		(property "Footprint" "Connector_JST:JST_SH_BM04B-SRSS-TB_1x04-1MP_P1.00mm_Vertical"
+		(property "Footprint" "Connector_JST:JST_SH_SM04B-SRSS-TB_1x04-1MP_P1.00mm_Horizontal"
 			(at 46.99 219.71 0)
 			(effects
@@
 			)
 		)
-		(property "Footprint" "Connector_JST:JST_SH_BM04B-SRSS-TB_1x04-1MP_P1.00mm_Vertical"
+		(property "Footprint" "Connector_JST:JST_SH_SM04B-SRSS-TB_1x04-1MP_P1.00mm_Horizontal"
 			(at 48.26 292.1 0)
 			(effects
