File: board/oval_v5.kicad_sch (KiCad schematic)
At the start: 147 parts, among them J1 HDR-5x1, J10 HDR-4x1, J11 HDR-4x1, J12 HDR-4x1, J13 HDR-4x1, J14 HDR-4x1, J15 HDR-4x1, J16 HDR-4x1, J17 HDR-4x1, J18 Conn_Coaxial, J19 Conn_01x02, J2 HDR-4x1, J20 Conn_01x02, J21 Conn_02x02_Counter_Clockwise, J22 HDR-2x1, J23 HDR-2x1, J25 Conn_01x06, J3 HDR-4x1, J4 Conn_01x06, J5 Micro_SD_Card, J6 Conn_01x02, J7 HDR-4x1, J8 Conn_01x08, J9 HDR-4x1, P1 USB_C_Plug_USB2.0, Q1 Q_PMOS_GSD, Q2 MMBT3904, Q3 MMBT3904, SW1 SW_DIP_x02, SW2 SW_DIP_x02, U1 RV-8803, U10 SiP32431DR3, U11 SiP32431DR3, U12 SiP32431DR3, U13 SiP32431DR3, U14 SiP32431DR3, U16 PCA9548APW, U17 SiP32431DR3, U18 PCA9555PW, U2 ESP32-S3-WROOM-1, U3 TMP117xxDRV, U4 RFM95W-915S2, U7 MAX3485, U8 AP7361C-33E, U9 AP7361C-33E

Commit message: working on board
Connections:
- net SCL_0: now also J15.4
- net SCL_1: now also J14.4
- net SCL_6: no longer J14.4
- net SCL_7: no longer J15.4
- net SDA_0: now also J15.3
- net SDA_1: now also J14.3
- net SDA_6: no longer J14.3
- net SDA_7: no longer J15.3
Other:
- moved on the sheet: D10
Changed lines of the file:
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@@
 	(text "OLD sensors\n"
 		(exclude_from_sim no)
-		(at 295.148 363.474 0)
+		(at 278.13 363.22 0)
 		(effects
 			(font
@@
 	(wire
 		(pts
-			(xy 306.07 441.96) (xy 306.07 440.69)
+			(xy 320.04 440.69) (xy 320.04 439.42)
 		)
 		(stroke
@@
 	(wire
 		(pts
-			(xy 304.8 422.91) (xy 306.07 422.91)
+			(xy 318.77 421.64) (xy 320.04 421.64)
 		)
 		(stroke
@@
 	(wire
 		(pts
-			(xy 306.07 422.91) (xy 306.07 425.45)
+			(xy 320.04 421.64) (xy 320.04 424.18)
 		)
 		(stroke
@@
 		)
 	)
-	(global_label "SDA_6"
+	(global_label "SDA_1"
 		(shape input)
 		(at 532.13 227.33 180)
@@
 	(global_label "RGB"
 		(shape input)
-		(at 298.45 433.07 180)
+		(at 312.42 431.8 180)
 		(fields_autoplaced yes)
 		(effects
@@
 		)
 		(property "Intersheetrefs" "${INTERSHEET_REFS}"
-			(at 291.6548 433.07 0)
+			(at 305.6248 431.8 0)
 			(effects
 				(font
@@
 		)
 	)
-	(global_label "SCL_6"
+	(global_label "SCL_1"
 		(shape input)
 		(at 532.13 229.87 180)
@@
 	(global_label "V_S1"
 		(shape input)
-		(at 304.8 422.91 180)
+		(at 318.77 421.64 180)
 		(fields_autoplaced yes)
 		(effects
@@
 		)
 		(property "Intersheetrefs" "${INTERSHEET_REFS}"
-			(at 297.3396 422.91 0)
+			(at 311.3096 421.64 0)
 			(effects
 				(font
@@
 		)
 	)
-	(global_label "SDA_7"
+	(global_label "SDA_0"
 		(shape input)
 		(at 532.13 247.65 180)
@@
 		)
 	)
-	(global_label "SCL_7"
+	(global_label "SCL_0"
 		(shape input)
 		(at 532.13 250.19 180)
@@
 	(symbol
 		(lib_id "power:GND")
-		(at 306.07 441.96 0)
+		(at 320.04 440.69 0)
 		(mirror y)
 		(unit 1)
@@
 		(dnp no)
 		(property "Reference" "#PWR067"
-			(at 306.07 448.31 0)
+			(at 320.04 447.04 0)
 			(effects
 				(font
@@
 		)
 		(property "Value" "GND"
-			(at 305.943 446.3542 0)
+			(at 319.913 445.0842 0)
 			(effects
 				(font
@@
 		)
 		(property "Footprint" ""
-			(at 306.07 441.96 0)
+			(at 320.04 440.69 0)
 			(effects
 				(font
@@
 		)
 		(property "Datasheet" ""
-			(at 306.07 441.96 0)
+			(at 320.04 440.69 0)
 			(effects
 				(font
@@
 		)
 		(property "Description" ""
-			(at 306.07 441.96 0)
+			(at 320.04 440.69 0)
 			(effects
 				(font
@@
 	(symbol
 		(lib_id "LED:WS2812B")
-		(at 306.07 433.07 0)
+		(at 320.04 431.8 0)
 		(unit 1)
 		(exclude_from_sim no)
@@
 		(fields_autoplaced yes)
 		(property "Reference" "D10"
-			(at 317.5 426.6498 0)
+			(at 331.47 425.3798 0)
 			(effects
 				(font
@@
 		)
 		(property "Value" "WS2812B"
-			(at 317.5 429.1898 0)
+			(at 331.47 427.9198 0)
 			(effects
 				(font
@@
 		)
 		(property "Footprint" "LED_SMD:LED_WS2812B_PLCC4_5.0x5.0mm_P3.2mm"
-			(at 307.34 440.69 0)
+			(at 321.31 439.42 0)
 			(effects
 				(font
@@
 		)
 		(property "Datasheet" "https://cdn-shop.adafruit.com/datasheets/WS2812B.pdf"
-			(at 308.61 442.595 0)
+			(at 322.58 441.325 0)
 			(effects
 				(font
@@
 		)
 		(property "Description" "RGB LED with integrated controller"
-			(at 306.07 433.07 0)
+			(at 320.04 431.8 0)
 			(effects
 				(font
